Commit message: all the final check of Motoman before creating new scenarios

File: motoman.urdf (robot description, URDF)
Before this commit: robot sda10f, 22 links, 21 joints
Joints:
- joint motoman_right_joint_pre_ee: origin xyz=0 0 -0.0 rpy=3.141 0 0 -> xyz=0 0 -0.035 rpy=3.141 0 0
- joint torso_joint_0: axis 0 0 1 -> (none); limit lower=-2.9570 upper=2.9570 effort=100 velocity=2.26 -> (none); type revolute -> fixed
